Commit message: version

File: description/robot_core.xacro (robot description, xacro)
@@ -1,16 +1,4 @@
 <?xml version="1.0"?>
 <robot xmlns:xacro="http://www.ros.org/wiki/xacro">
-    <material name="white">
-        <color rgba="1 1 1 1"/>
-    </material>
-    <material name="orange">
-        <color rgba="1 0.3 0.1 1"/>
-    </material>
-    <material name="blue">
-        <color rgba="0.2 0.2 1 1"/>
-    </material>
-    <material name="black">
-        <color rgba="0 0 0 1"/>
-    </material>
     <link name="base_link">
     </link>

Commit message: version

File: description/robot_core.xacro (robot description, xacro)
@@ -1,4 +1,16 @@
 <?xml version="1.0"?>
 <robot xmlns:xacro="http://www.ros.org/wiki/xacro">
+    <material name="white">
+        <color rgba="1 1 1 1"/>
+    </material>
+    <material name="orange">
+        <color rgba="1 0.3 0.1 1"/>
+    </material>
+    <material name="blue">
+        <color rgba="0.2 0.2 1 1"/>
+    </material>
+    <material name="black">
+        <color rgba="0 0 0 1"/>
+    </material>
     <link name="base_link">
     </link>

Commit message: modify Links

File: description/robot_core.xacro (robot description, xacro)
@@ -20,4 +20,5 @@
         <origin xyz="-0.1 0 0"/>
     </joint>
+    <!-- CHASSIS -->
     <link name="chassis">
         <visual>
@@ -28,4 +29,14 @@
             <material name="white"/>
         </visual>
+        <collision>
+            <origin xyz="0.10 0 0.07" rpy="0 0 0"/>
+            <geometry>
+                <box size="0.20 0.19 0.12"/>
+            </geometry>
+        </collision>
+        <!-- ... intertia ... -->
+        <xacro:inertial_box mass="0.5" x="0.20" y="0.19" z="0.12">
+            <origin xyz="0.15 0 0.075" rpy="0 0 0"/>
+        </xacro:inertial_box>
     </link>
     <!-- LEFT BACK WHEEL -->
@@ -43,4 +54,8 @@
             <material name="blue"/>
         </visual>
+        <!-- ... visual and collision here ... -->
+        <xacro:inertial_cylinder mass="0.1" length="0.035" radius="0.06">
+            <origin xyz="0 0 0" rpy="0 0 0"/>
+        </xacro:inertial_cylinder>
     </link>
     <!-- RIGHT BACK WHEEL -->
@@ -58,4 +73,8 @@
             <material name="blue"/>
         </visual>
+        <!-- ... visual and collision here ... -->
+        <xacro:inertial_cylinder mass="0.1" length="0.035" radius="0.06">
+            <origin xyz="0 0 0" rpy="0 0 0"/>
+        </xacro:inertial_cylinder>
     </link>
     <!-- LEFT FRONT WHEEL -->
@@ -73,4 +92,8 @@
             <material name="blue"/>
         </visual>
+        <!-- ... visual and collision here ... -->
+        <xacro:inertial_cylinder mass="0.1" length="0.035" radius="0.06">
+            <origin xyz="0 0 0" rpy="0 0 0"/>
+        </xacro:inertial_cylinder>
     </link>
     <!-- RIGHT FRONT WHEEL -->
@@ -88,50 +111,4 @@
             <material name="blue"/>
         </visual>
-    </link>
-    <link name="chassis">
-        <visual>
-            <origin xyz="0.10 0 0.07" rpy="0 0 0"/>
-            <geometry>
-                <box size="0.20 0.19 0.12"/>
-            </geometry>
-            <material name="white"/>
-        </visual>
-        <collision>
-            <origin xyz="0.10 0 0.07" rpy="0 0 0"/>
-            <geometry>
-                <box size="0.20 0.19 0.12"/>
-            </geometry>
-        </collision>
-    </link>
-    <!-- ... intertia ... -->
-    <link name="chassis">
-        <!-- ... visual and collision here ... -->
-        <xacro:inertial_box mass="0.5" x="0.20" y="0.19" z="0.12">
-            <origin xyz="0.15 0 0.075" rpy="0 0 0"/>
-        </xacro:inertial_box>
-    </link>
-    <!-- left front wheel inertia -->
-    <link name="left_front_wheel">
-        <!-- ... visual and collision here ... -->
-        <xacro:inertial_cylinder mass="0.1" length="0.035" radius="0.06">
-            <origin xyz="0 0 0" rpy="0 0 0"/>
-        </xacro:inertial_cylinder>
-    </link>
-    <!-- Right front wheel inertia -->
-    <link name="right_front_wheel">
-        <!-- ... visual and collision here ... -->
-        <xacro:inertial_cylinder mass="0.1" length="0.035" radius="0.06">
-            <origin xyz="0 0 0" rpy="0 0 0"/>
-        </xacro:inertial_cylinder>
-    </link>
-    <!-- left back wheel inertia -->
-    <link name="left_back_wheel">
-        <!-- ... visual and collision here ... -->
-        <xacro:inertial_cylinder mass="0.1" length="0.035" radius="0.06">
-            <origin xyz="0 0 0" rpy="0 0 0"/>
-        </xacro:inertial_cylinder>
-    </link>
-    <!-- Right back wheel inertia -->
-    <link name="right_back_wheel">
         <!-- ... visual and collision here ... -->
         <xacro:inertial_cylinder mass="0.1" length="0.035" radius="0.06">

Commit message: modif local viz OK test

File: description/robot_core.xacro (robot description, xacro)
@@ -100,5 +100,5 @@
             <material name="blue"/>
         </visual>
-		<collision>
+        <collision>
             <geometry>
                 <cylinder radius="0.035" length="0.06"/>

Commit message: modif local viz OK test

File: description/robot_core.xacro (robot description, xacro)
@@ -23,9 +23,5 @@
     <link name="chassis">
         <visual>
-<<<<<<< HEAD
             <origin xyz="0.10 0 0.035" rpy="0 0 0"/>
-=======
-            <origin xyz="0.10 0 0.07" rpy="0 0 0"/>
->>>>>>> a857f3169a5c65cf19696927df2dc6cf8b4c78b2
             <geometry>
                 <box size="0.20 0.19 0.12"/>
@@ -34,9 +30,5 @@
         </visual>
         <collision>
-<<<<<<< HEAD
             <origin xyz="0.10 0 0.035" rpy="0 0 0"/>
-=======
-            <origin xyz="0.10 0 0.07" rpy="0 0 0"/>
->>>>>>> a857f3169a5c65cf19696927df2dc6cf8b4c78b2
             <geometry>
                 <box size="0.20 0.19 0.12"/>
@@ -51,18 +43,11 @@
     <joint name="left_back_wheel_joint" type="continuous">
         <parent link="base_link"/>
-<<<<<<< HEAD
         <child link="left_back_wheel"/>
         <origin xyz="-0.0675 0.09 0" rpy="${pi/2} 0 0" />
         <axis xyz="0 0 -1"/>
-=======
-        <child link="left_wheel"/>
-        <origin xyz="-0.0675 0.09 0" rpy="-${pi/2} 0 0"/>
-        <axis xyz="0 0 1"/>
->>>>>>> a857f3169a5c65cf19696927df2dc6cf8b4c78b2
     </joint>
     <link name="left_back_wheel">
         <visual>
             <geometry>
-<<<<<<< HEAD
                 <cylinder radius="0.035" length="0.06"/>
             </geometry>
@@ -74,11 +59,4 @@
             </geometry>
         </collision>
-=======
-                <cylinder length="0.035" radius="0.06" />/>
-            </geometry>
-            <material name="blue"/>
-        </visual>
-        <!-- ... visual and collision here ... -->
->>>>>>> a857f3169a5c65cf19696927df2dc6cf8b4c78b2
         <xacro:inertial_cylinder mass="0.1" length="0.035" radius="0.06">
             <origin xyz="0 0 0" rpy="0 0 0"/>
@@ -88,9 +66,5 @@
     <joint name="right_back_wheel_joint" type="continuous">
         <parent link="base_link"/>
-<<<<<<< HEAD
         <child link="right_back_wheel"/>
-=======
-        <child link="right_wheel"/>
->>>>>>> a857f3169a5c65cf19696927df2dc6cf8b4c78b2
         <origin xyz="-0.0675 -0.09 0" rpy="${pi/2} 0 0"/>
         <axis xyz="0 0 -1"/>
@@ -99,5 +73,4 @@
         <visual>
             <geometry>
-<<<<<<< HEAD
                 <cylinder radius="0.035" length="0.06" />/>
             </geometry>
@@ -109,11 +82,4 @@
             </geometry>
         </collision>
-=======
-                <cylinder length="0.035" radius="0.06" />/>
-            </geometry>
-            <material name="blue"/>
-        </visual>
-        <!-- ... visual and collision here ... -->
->>>>>>> a857f3169a5c65cf19696927df2dc6cf8b4c78b2
         <xacro:inertial_cylinder mass="0.1" length="0.035" radius="0.06">
             <origin xyz="0 0 0" rpy="0 0 0"/>
@@ -123,9 +89,5 @@
     <joint name="left_front_wheel_joint" type="continuous">
         <parent link="base_link"/>
-<<<<<<< HEAD
         <child link="left_front_wheel"/>
-=======
-        <child link="left_wheel"/>
->>>>>>> a857f3169a5c65cf19696927df2dc6cf8b4c78b2
         <origin xyz="0.0675 0.09 0" rpy="-${pi/2} 0 0"/>
         <axis xyz="0 0 1"/>
@@ -134,5 +96,4 @@
         <visual>
             <geometry>
-<<<<<<< HEAD
                 <cylinder radius="0.035" length="0.06" />/>
             </geometry>
@@ -144,11 +105,4 @@
             </geometry>
         </collision>
-=======
-                <cylinder length="0.035" radius="0.06" />/>
-            </geometry>
-            <material name="blue"/>
-        </visual>
-        <!-- ... visual and collision here ... -->
->>>>>>> a857f3169a5c65cf19696927df2dc6cf8b4c78b2
         <xacro:inertial_cylinder mass="0.1" length="0.035" radius="0.06">
             <origin xyz="0 0 0" rpy="0 0 0"/>
@@ -158,9 +112,5 @@
     <joint name="right_front_wheel_joint" type="continuous">
         <parent link="base_link"/>
-<<<<<<< HEAD
         <child link="right_front_wheel"/>
-=======
-        <child link="right_wheel"/>
->>>>>>> a857f3169a5c65cf19696927df2dc6cf8b4c78b2
         <origin xyz="0.0675 -0.09 0" rpy="${pi/2} 0 0"/>
         <axis xyz="0 0 -1"/>
@@ -169,5 +119,4 @@
         <visual>
             <geometry>
-<<<<<<< HEAD
                 <cylinder radius="0.035" length="0.06" />/>
             </geometry>
@@ -179,18 +128,7 @@
             </geometry>
         </collision>
-=======
-                <cylinder length="0.035" radius="0.06" />/>
-            </geometry>
-            <material name="blue"/>
-        </visual>
-        <!-- ... visual and collision here ... -->
->>>>>>> a857f3169a5c65cf19696927df2dc6cf8b4c78b2
         <xacro:inertial_cylinder mass="0.1" length="0.035" radius="0.06">
             <origin xyz="0 0 0" rpy="0 0 0"/>
         </xacro:inertial_cylinder>
     </link>
-<<<<<<< HEAD
 </robot>
-=======
-</robot>
->>>>>>> a857f3169a5c65cf19696927df2dc6cf8b4c78b2

Commit message: modif local pour merge

File: description/robot_core.xacro (robot description, xacro)
@@ -59,4 +59,5 @@
             </geometry>
         </collision>
+        <!-- ... intertia ... -->
         <xacro:inertial_cylinder mass="0.1" length="0.035" radius="0.06">
             <origin xyz="0 0 0" rpy="0 0 0"/>
@@ -77,9 +78,10 @@
             <material name="blue"/>
         </visual>
-		<collision>
+        <collision>
             <geometry>
                 <cylinder radius="0.035" length="0.06"/>
             </geometry>
         </collision>
+        <!-- ... intertia ... -->
         <xacro:inertial_cylinder mass="0.1" length="0.035" radius="0.06">
             <origin xyz="0 0 0" rpy="0 0 0"/>
@@ -105,4 +107,5 @@
             </geometry>
         </collision>
+		<!-- ... intertia ... -->
         <xacro:inertial_cylinder mass="0.1" length="0.035" radius="0.06">
             <origin xyz="0 0 0" rpy="0 0 0"/>
@@ -128,4 +131,5 @@
             </geometry>
         </collision>
+        <!-- ... intertia ... -->
         <xacro:inertial_cylinder mass="0.1" length="0.035" radius="0.06">
             <origin xyz="0 0 0" rpy="0 0 0"/>

Commit message: add lidar to urdf

File: description/robot_core.xacro (robot description, xacro)
@@ -44,6 +44,6 @@
         <parent link="base_link"/>
         <child link="left_back_wheel"/>
-        <origin xyz="-0.0675 0.09 0" rpy="${pi/2} 0 0" />
-        <axis xyz="0 0 -1"/>
+        <origin xyz="-0.0675 0.08 0" rpy="-${pi/2} 0 0" />
+        <axis xyz="0 0 1"/>
     </joint>
     <link name="left_back_wheel">
@@ -64,9 +64,33 @@
         </xacro:inertial_cylinder>
     </link>
+    <!-- LEFT FRONT WHEEL -->
+    <joint name="left_front_wheel_joint" type="continuous">
+        <parent link="base_link"/>
+        <child link="left_front_wheel"/>
+        <origin xyz="0.0675 0.08 0" rpy="-${pi/2} 0 0"/>
+        <axis xyz="0 0 1"/>
+    </joint>
+    <link name="left_front_wheel">
+        <visual>
+            <geometry>
+                <cylinder radius="0.035" length="0.06" />/>
+            </geometry>
+            <material name="blue"/>
+        </visual>
+        <collision>
+            <geometry>
+                <cylinder radius="0.035" length="0.06"/>
+            </geometry>
+        </collision>
+		<!-- ... intertia ... -->
+        <xacro:inertial_cylinder mass="0.1" length="0.035" radius="0.06">
+            <origin xyz="0 0 0" rpy="0 0 0"/>
+        </xacro:inertial_cylinder>
+    </link>
     <!-- RIGHT BACK WHEEL -->
     <joint name="right_back_wheel_joint" type="continuous">
         <parent link="base_link"/>
         <child link="right_back_wheel"/>
-        <origin xyz="-0.0675 -0.09 0" rpy="${pi/2} 0 0"/>
+        <origin xyz="-0.0675 -0.08 0" rpy="${pi/2} 0 0"/>
         <axis xyz="0 0 -1"/>
     </joint>
@@ -88,33 +112,9 @@
         </xacro:inertial_cylinder>
     </link>
-    <!-- LEFT FRONT WHEEL -->
-    <joint name="left_front_wheel_joint" type="continuous">
-        <parent link="base_link"/>
-        <child link="left_front_wheel"/>
-        <origin xyz="0.0675 0.09 0" rpy="-${pi/2} 0 0"/>
-        <axis xyz="0 0 1"/>
-    </joint>
-    <link name="left_front_wheel">
-        <visual>
-            <geometry>
-                <cylinder radius="0.035" length="0.06" />/>
-            </geometry>
-            <material name="blue"/>
-        </visual>
-        <collision>
-            <geometry>
-                <cylinder radius="0.035" length="0.06"/>
-            </geometry>
-        </collision>
-		<!-- ... intertia ... -->
-        <xacro:inertial_cylinder mass="0.1" length="0.035" radius="0.06">
-            <origin xyz="0 0 0" rpy="0 0 0"/>
-        </xacro:inertial_cylinder>
-    </link>
     <!-- RIGHT FRONT WHEEL -->
     <joint name="right_front_wheel_joint" type="continuous">
         <parent link="base_link"/>
         <child link="right_front_wheel"/>
-        <origin xyz="0.0675 -0.09 0" rpy="${pi/2} 0 0"/>
+        <origin xyz="0.0675 -0.08 0" rpy="${pi/2} 0 0"/>
         <axis xyz="0 0 -1"/>
     </joint>
@@ -136,3 +136,27 @@
         </xacro:inertial_cylinder>
     </link>
+    <!-- LIDAR -->
+    <joint name="lidar_joint" type="fixed">
+        <parent link="chassis"/>
+        <child link="lidar"/>
+        <origin xyz="0.08 0 0.10" rpy="0 0 0"/>
+        <axis xyz="0 0 0"/>
+    </joint>
+    <link name="lidar">
+        <visual>
+            <geometry>
+                <cylinder radius="0.035" length="0.06" />/>
+            </geometry>
+            <material name="black"/>
+        </visual>
+        <collision>
+            <geometry>
+                <cylinder radius="0.035" length="0.06"/>
+            </geometry>
+        </collision>
+        <!-- ... intertia ... -->
+        <xacro:inertial_cylinder mass="0.1" length="0.035" radius="0.06">
+            <origin xyz="0 0 0" rpy="0 0 0"/>
+        </xacro:inertial_cylinder>
+    </link>
 </robot>
