Commit message: rename LidarBot to lidar_bot

File: description/robot.urdf.xacro (robot description, xacro)
@@ -3,3 +3,4 @@
     <!-- Example link -->
     <xacro:include filename="robot_core.xacro" />
+    <xacro:include filename="inertial_macros.xacro" />
 </robot>

File: description/robot_core.xacro (robot description, xacro)
@@ -15,3 +15,127 @@
     <link name="base_link">
     </link>
+    <joint name="chassis_joint" type="fixed">
+        <parent link="base_link"/>
+        <child link="chassis"/>
+        <origin xyz="-0.1 0 0"/>
+    </joint>
+    <link name="chassis">
+        <visual>
+            <origin xyz="0.10 0 0.07" rpy="0 0 0"/>
+            <geometry>
+                <box size="0.20 0.19 0.12"/>
+            </geometry>
+            <material name="white"/>
+        </visual>
+    </link>
+    <!-- LEFT BACK WHEEL -->
+    <joint name="left_back_wheel_joint" type="continuous">
+        <parent link="base_link"/>
+        <child link="left_wheel"/>
+        <origin xyz="-0.0675 0.09 0" rpy="-${pi/2} 0 0"/>
+        <axis xyz="0 0 1"/>
+    </joint>
+    <link name="left_back_wheel">
+        <visual>
+            <geometry>
+                <cylinder length="0.035" radius="0.06" />/>
+            </geometry>
+            <material name="blue"/>
+        </visual>
+    </link>
+    <!-- RIGHT BACK WHEEL -->
+    <joint name="right_back_wheel_joint" type="continuous">
+        <parent link="base_link"/>
+        <child link="right_wheel"/>
+        <origin xyz="-0.0675 -0.09 0" rpy="${pi/2} 0 0"/>
+        <axis xyz="0 0 -1"/>
+    </joint>
+    <link name="right_back_wheel">
+        <visual>
+            <geometry>
+                <cylinder length="0.035" radius="0.06" />/>
+            </geometry>
+            <material name="blue"/>
+        </visual>
+    </link>
+    <!-- LEFT FRONT WHEEL -->
+    <joint name="left_front_wheel_joint" type="continuous">
+        <parent link="base_link"/>
+        <child link="left_wheel"/>
+        <origin xyz="0.0675 0.09 0" rpy="-${pi/2} 0 0"/>
+        <axis xyz="0 0 1"/>
+    </joint>
+    <link name="left_front_wheel">
+        <visual>
+            <geometry>
+                <cylinder length="0.035" radius="0.06" />/>
+            </geometry>
+            <material name="blue"/>
+        </visual>
+    </link>
+    <!-- RIGHT FRONT WHEEL -->
+    <joint name="right_front_wheel_joint" type="continuous">
+        <parent link="base_link"/>
+        <child link="right_wheel"/>
+        <origin xyz="0.0675 -0.09 0" rpy="${pi/2} 0 0"/>
+        <axis xyz="0 0 -1"/>
+    </joint>
+    <link name="right_front_wheel">
+        <visual>
+            <geometry>
+                <cylinder length="0.035" radius="0.06" />/>
+            </geometry>
+            <material name="blue"/>
+        </visual>
+    </link>
+    <link name="chassis">
+        <visual>
+            <origin xyz="0.10 0 0.07" rpy="0 0 0"/>
+            <geometry>
+                <box size="0.20 0.19 0.12"/>
+            </geometry>
+            <material name="white"/>
+        </visual>
+        <collision>
+            <origin xyz="0.10 0 0.07" rpy="0 0 0"/>
+            <geometry>
+                <box size="0.20 0.19 0.12"/>
+            </geometry>
+        </collision>
+    </link>
+    <!-- ... intertia ... -->
+    <link name="chassis">
+        <!-- ... visual and collision here ... -->
+        <xacro:inertial_box mass="0.5" x="0.20" y="0.19" z="0.12">
+            <origin xyz="0.15 0 0.075" rpy="0 0 0"/>
+        </xacro:inertial_box>
+    </link>
+    <!-- left front wheel inertia -->
+    <link name="left_front_wheel">
+        <!-- ... visual and collision here ... -->
+        <xacro:inertial_cylinder mass="0.1" length="0.035" radius="0.06">
+            <origin xyz="0 0 0" rpy="0 0 0"/>
+        </xacro:inertial_cylinder>
+    </link>
+    <!-- Right front wheel inertia -->
+    <link name="right_front_wheel">
+        <!-- ... visual and collision here ... -->
+        <xacro:inertial_cylinder mass="0.1" length="0.035" radius="0.06">
+            <origin xyz="0 0 0" rpy="0 0 0"/>
+        </xacro:inertial_cylinder>
+    </link>
+    <!-- left back wheel inertia -->
+    <link name="left_back_wheel">
+        <!-- ... visual and collision here ... -->
+        <xacro:inertial_cylinder mass="0.1" length="0.035" radius="0.06">
+            <origin xyz="0 0 0" rpy="0 0 0"/>
+        </xacro:inertial_cylinder>
+    </link>
+    <!-- Right back wheel inertia -->
+    <link name="right_back_wheel">
+        <!-- ... visual and collision here ... -->
+        <xacro:inertial_cylinder mass="0.1" length="0.035" radius="0.06">
+            <origin xyz="0 0 0" rpy="0 0 0"/>
+        </xacro:inertial_cylinder>
+    </link>
 </robot>

Commit message: add delta2g and camera

File: description/robot.urdf.xacro (robot description, xacro)
@@ -4,3 +4,6 @@
     <xacro:include filename="inertial_macros.xacro" />
     <xacro:include filename="robot_core.xacro" />
+	<xacro:include filename="gazebo_control.xacro" />
+	<xacro:include filename="lidar.xacro" />
+	<xacro:include filename="camera.xacro" />
 </robot>

File: description/robot_core.xacro (robot description, xacro)
@@ -13,4 +13,7 @@
         <color rgba="0 0 0 1"/>
     </material>
+	<material name="red">
+		<color rgba="1 0 0 1"/>
+	</material>
     <link name="base_link">
     </link>
@@ -25,5 +28,5 @@
             <origin xyz="0.10 0 0.035" rpy="0 0 0"/>
             <geometry>
-                <box size="0.20 0.19 0.12"/>
+                <box size="0.20 0.19 0.13"/>
             </geometry>
             <material name="white"/>
@@ -32,13 +35,16 @@
             <origin xyz="0.10 0 0.035" rpy="0 0 0"/>
             <geometry>
-                <box size="0.20 0.19 0.12"/>
+                <box size="0.20 0.19 0.13"/>
             </geometry>
         </collision>
         <!-- ... intertia ... -->
-        <xacro:inertial_box mass="0.5" x="0.20" y="0.19" z="0.12">
+        <xacro:inertial_box mass="0.5" x="0.20" y="0.19" z="0.13">
             <origin xyz="0.15 0 0.075" rpy="0 0 0"/>
         </xacro:inertial_box>
     </link>
-    <!-- LEFT BACK WHEEL -->
+	<gazebo reference="chassis">
+		<material>Gazebo/White</material>
+	</gazebo>
+	<!-- LEFT BACK WHEEL -->
     <joint name="left_back_wheel_joint" type="continuous">
         <parent link="base_link"/>
@@ -64,4 +70,7 @@
         </xacro:inertial_cylinder>
     </link>
+	<gazebo reference="left_back_wheel">
+		<material>Gazebo/Blue</material>
+	</gazebo>
     <!-- LEFT FRONT WHEEL -->
     <joint name="left_front_wheel_joint" type="continuous">
@@ -74,5 +83,5 @@
         <visual>
             <geometry>
-                <cylinder radius="0.035" length="0.06" />/>
+                <cylinder radius="0.035" length="0.06" />
             </geometry>
             <material name="blue"/>
@@ -88,4 +97,9 @@
         </xacro:inertial_cylinder>
     </link>
+	<gazebo reference="left_front_wheel">
+		<material>Gazebo/Blue</material>
+		<mu1 value="0.1"/>
+		<mu2 value="0.1"/>
+	</gazebo>
     <!-- RIGHT BACK WHEEL -->
     <joint name="right_back_wheel_joint" type="continuous">
@@ -98,5 +112,5 @@
         <visual>
             <geometry>
-                <cylinder radius="0.035" length="0.06" />/>
+                <cylinder radius="0.035" length="0.06" />
             </geometry>
             <material name="blue"/>
@@ -112,4 +126,7 @@
         </xacro:inertial_cylinder>
     </link>
+	<gazebo reference="right_back_wheel">
+		<material>Gazebo/Blue</material>
+	</gazebo>
     <!-- RIGHT FRONT WHEEL -->
     <joint name="right_front_wheel_joint" type="continuous">
@@ -122,5 +139,5 @@
         <visual>
             <geometry>
-                <cylinder radius="0.035" length="0.06" />/>
+                <cylinder radius="0.035" length="0.06" />
             </geometry>
             <material name="blue"/>
@@ -136,27 +153,8 @@
         </xacro:inertial_cylinder>
     </link>
-    <!-- LIDAR -->
-    <joint name="lidar_joint" type="fixed">
-        <parent link="chassis"/>
-        <child link="lidar"/>
-        <origin xyz="0.08 0 0.10" rpy="0 0 0"/>
-        <axis xyz="0 0 0"/>
-    </joint>
-    <link name="lidar">
-        <visual>
-            <geometry>
-                <cylinder radius="0.035" length="0.06" />/>
-            </geometry>
-            <material name="black"/>
-        </visual>
-        <collision>
-            <geometry>
-                <cylinder radius="0.035" length="0.06"/>
-            </geometry>
-        </collision>
-        <!-- ... intertia ... -->
-        <xacro:inertial_cylinder mass="0.1" length="0.035" radius="0.06">
-            <origin xyz="0 0 0" rpy="0 0 0"/>
-        </xacro:inertial_cylinder>
-    </link>
+	<gazebo reference="right_front_wheel">
+		<material>Gazebo/Blue</material>
+		<mu1 value="0.1"/>
+		<mu2 value="0.1"/>
+	</gazebo>
 </robot>
