Commit message: Add camera

File: description/lidar.xacro (robot description, xacro)
@@ -9,5 +9,5 @@
     <link name="delta2g">
         <visual>
-			<origin xyz="0 0 -0.05" rpy="0 0 0"/>
+			<origin xyz="0 0 -0.05" rpy="0 0 ${pi}"/>
             <geometry>
                 <cylinder radius="0.035" length="0.06" />
@@ -16,9 +16,12 @@
         </visual>
     </link>
+	<gazebo reference="delta2g">
+		<material>Gazebo/Black</material>
+	</gazebo>
 	 <!-- LIDAR -->
     <joint name="lidar_joint" type="fixed">
         <parent link="chassis"/>
         <child link="lidar"/>
-        <origin xyz="0.06 0 0.18" rpy="0 0 0"/>
+        <origin xyz="0.06 0 0.20" rpy="0 0 0"/>
     </joint>
     <link name="lidar">

File: description/robot.urdf.xacro (robot description, xacro)
@@ -1,8 +1,14 @@
 <?xml version="1.0"?>
 <robot xmlns:xacro="http://www.ros.org/wiki/xacro"  name="lidar_bot">
+	<xacro:arg name="use_ros2_control" default="true"/>
     <!-- Example link -->
     <xacro:include filename="inertial_macros.xacro" />
     <xacro:include filename="robot_core.xacro" />
-	<xacro:include filename="gazebo_control.xacro" />
+	<xacro:if value="$(arg use_ros2_control)">
+		<xacro:include filename="ros2_control.xacro" />
+	</xacro:if>
+	<xacro:unless value="$(arg use_ros2_control)">
+		<xacro:include filename="gazebo_control.xacro" />
+	</xacro:unless>
 	<xacro:include filename="lidar.xacro" />
 	<xacro:include filename="camera.xacro" />

File: description/robot_core.xacro (robot description, xacro)
@@ -62,5 +62,6 @@
         <collision>
             <geometry>
-                <cylinder radius="0.035" length="0.06"/>
+                <!-- <cylinder radius="0.035" length="0.06"/> -->
+                <sphere  radius="0.035"/>
             </geometry>
         </collision>
@@ -74,6 +75,6 @@
 	</gazebo>
     <!-- LEFT FRONT WHEEL -->
-    <joint name="left_front_wheel_joint" type="continuous">
-        <parent link="base_link"/>
+    <joint name="left_front_wheel_joint" type="continuous"> <!--   continuous -->
+        <parent link="base_link"/> <!--   base_link -->
         <child link="left_front_wheel"/>
         <origin xyz="0.0675 0.08 0" rpy="-${pi/2} 0 0"/>
@@ -118,6 +119,7 @@
         <collision>
             <geometry>
-                <cylinder radius="0.035" length="0.06"/>
-            </geometry>
+                <!-- <cylinder radius="0.035" length="0.06"/> -->
+                <sphere  radius="0.035"/>
+			</geometry>
         </collision>
         <!-- ... intertia ... -->
@@ -130,6 +132,6 @@
 	</gazebo>
     <!-- RIGHT FRONT WHEEL -->
-    <joint name="right_front_wheel_joint" type="continuous">
-        <parent link="base_link"/>
+    <joint name="right_front_wheel_joint" type="continuous">  <!--   continuous -->
+        <parent link="base_link"/>  <!--   base_link -->
         <child link="right_front_wheel"/>
         <origin xyz="0.0675 -0.08 0" rpy="${pi/2} 0 0"/>
